File: PCB/BellWAGO/Bell.kicad_pcb (KiCad board)
At the start: 2 copper layers, 70 x 70 mm, 50 parts, among them J1 USB-C-Socket-V, J10 FAULT, J11 FAULT, J2 BL, J5 Conn_01x05, J7 BELL, J8 PWR, J9 PWR, U1 MD8942, U3 ISL89410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

Commit message: Overprint, and tidy
Parts:
- added AJK1: AJK, RevK:AJK, F.Cu at (109.4, 95.9)
- J11: value FAULT -> TAMP
- U6: value ESP32-S3-MINI-1 -> ESP32-S3-MINI-1-N4R2
- moved J1 0.47 mm to (86.0, 105.0)
Connections:
- J7 pad 1: ENGHOLD -> BELL
- J7 pad 3: BELL -> ENGHOLD
Routing:
- net BELL: track 30.2 -> 20.0 mm
- net STB: track 30.3 -> 31.0 mm
