File: PCB/BellWAGO/Bell.kicad_sch (KiCad schematic)
At the start: 51 parts, among them J1 USB-C-Socket-V, J10 FAULT, J11 FAULT, J2 BL, J5 Conn_01x05, J7 BELL, J8 PWR, J9 PWR, U1 MD8942, U3 ISL89410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

Commit message: Overprint, and tidy
Parts:
- D1, D10, V1, V2, V3, V4: value ~ -> (none)
- J10, J8, J9: symbol Connector_Generic:Conn_01x02 -> RevK:WAGO2
- J11: value FAULT -> TAMP; symbol Connector_Generic:Conn_01x02 -> RevK:WAGO2
- J2: symbol Connector_Generic:Conn_01x01 -> RevK:WAGO1
- J7: symbol Connector_Generic:Conn_01x03 -> RevK:WAGO3
Connections:
- net +12V: now also J8.2A (2), J9.2A (2)
- net BELL: now also J7.1, J7.1A (1); no longer J7.3 (Pin_3)
- net ENGHOLD: now also J7.3, J7.3A (3); no longer J7.1 (Pin_1)
- net FAULT: now also J10.2A (2)
- net GND: now also J10.1A (1), J11.1A (1), J8.1A (1), J9.1A (1)
- net STB: now also J7.2A (2)
- net T: now also J11.2A (2)
- net ~{BACKLIGHT}: now also J2.1A (1)
- no-connect marks 26 -> 28
Other:
- moved on the sheet: C8, R8, U6
